Commit message: 新dqn_60000結果

File: dynamics/src/dynamics/urdf/single_arm_v22_19cm.urdf (robot description, URDF)
Before this commit: robot single_arm_v22_19cm, 8 links, 7 joints
Links:
- link link2: mass 1.33974234835036 -> 1.4616991950496234
- link link3: mass 1.19767908022107 -> 1.1178444141286732
Joints:
- joint joint3: origin xyz=0.214867681425003 0 -0.039 rpy=0 0 0 -> xyz=0.3107134125235618 0 -0.039 rpy=0 0 0
- joint joint4: origin xyz=0.285132318574997 0 0.039 rpy=0 0 -3.14159265358979 -> xyz=0.22239035577643562 0 0.039 rpy=0 0 -3.14159265358979

File: dynamics/src/dynamics/urdf/single_arm_v22_19cm_motion.urdf (robot description, URDF)
Before this commit: robot single_arm_v22_19cm, 8 links, 7 joints
Links:
- link link2: mass 1.33974234835036 -> 1.4616991950496234
- link link3: mass 1.19767908022107 -> 1.1178444141286732
Joints:
- joint joint3: origin xyz=0.214867681425003 0 -0.039 rpy=0 0 0 -> xyz=0.3107134125235618 0 -0.039 rpy=0 0 0
- joint joint4: origin xyz=0.285132318574997 0 0.039 rpy=0 0 -3.14159265358979 -> xyz=0.22239035577643562 0 0.039 rpy=0 0 -3.14159265358979

Commit message: 0320-cmd-2

File: dynamics/src/dynamics/urdf/single_arm_v22_19cm.urdf (robot description, URDF)
Before this commit: robot single_arm_v22_19cm, 8 links, 7 joints
Links:
- link link2: mass 1.4616991950496234 -> 1.51331934678338
- link link3: mass 1.1178444141286732 -> 1.35493351035948
Joints:
- joint joint3: origin xyz=0.3107134125235618 0 -0.039 rpy=0 0 0 -> xyz=0.351281624282433 0 -0.039 rpy=0 0 0
- joint joint4: origin xyz=0.22239035577643562 0 0.039 rpy=0 0 -3.14159265358979 -> xyz=0.408718375717567 0 0.039 rpy=0 0 -3.14159265358979

File: dynamics/src/dynamics/urdf/single_arm_v22_19cm_motion.urdf (robot description, URDF)
Before this commit: robot single_arm_v22_19cm, 8 links, 7 joints
Links:
- link link2: mass 1.4616991950496234 -> 1.51331934678338
- link link3: mass 1.1178444141286732 -> 1.35493351035948
Joints:
- joint joint3: origin xyz=0.3107134125235618 0 -0.039 rpy=0 0 0 -> xyz=0.351281624282433 0 -0.039 rpy=0 0 0
- joint joint4: origin xyz=0.22239035577643562 0 0.039 rpy=0 0 -3.14159265358979 -> xyz=0.408718375717567 0 0.039 rpy=0 0 -3.14159265358979

Commit message: episode return

File: dynamics/src/dynamics/urdf/single_arm_v22_19cm.urdf (robot description, URDF)
Before this commit: robot single_arm_v22_19cm, 8 links, 7 joints
Links:
- link link2: mass 1.51331934678338 -> 1.3044239868593668
- link link3: mass 1.35493351035948 -> 1.2285446023550037
Joints:
- joint joint3: origin xyz=0.351281624282433 0 -0.039 rpy=0 0 0 -> xyz=0.18711102593640605 0 -0.039 rpy=0 0 0
- joint joint4: origin xyz=0.408718375717567 0 0.039 rpy=0 0 -3.14159265358979 -> xyz=0.30938949326204396 0 0.039 rpy=0 0 -3.14159265358979

File: dynamics/src/dynamics/urdf/single_arm_v22_19cm_motion.urdf (robot description, URDF)
Before this commit: robot single_arm_v22_19cm, 8 links, 7 joints
Links:
- link link2: mass 1.51331934678338 -> 1.3044239868593668
- link link3: mass 1.35493351035948 -> 1.2285446023550037
Joints:
- joint joint3: origin xyz=0.351281624282433 0 -0.039 rpy=0 0 0 -> xyz=0.18711102593640605 0 -0.039 rpy=0 0 0
- joint joint4: origin xyz=0.408718375717567 0 0.039 rpy=0 0 -3.14159265358979 -> xyz=0.30938949326204396 0 0.039 rpy=0 0 -3.14159265358979

Commit message: 0325_test

File: dynamics/src/dynamics/urdf/single_arm_v22_19cm.urdf (robot description, URDF)
Before this commit: robot single_arm_v22_19cm, 8 links, 7 joints
Links:
- link link2: mass 1.3044239868593668 -> 1.3205667282817466
- link link3: mass 1.2285446023550037 -> 1.0432921141432132
Joints:
- joint joint3: origin xyz=0.18711102593640605 0 -0.039 rpy=0 0 0 -> xyz=0.19979758594052155 0 -0.039 rpy=0 0 0
- joint joint4: origin xyz=0.30938949326204396 0 0.039 rpy=0 0 -3.14159265358979 -> xyz=0.16379979779976328 0 0.039 rpy=0 0 -3.14159265358979

File: dynamics/src/dynamics/urdf/single_arm_v22_19cm_motion.urdf (robot description, URDF)
Before this commit: robot single_arm_v22_19cm, 8 links, 7 joints
Links:
- link link2: mass 1.3044239868593668 -> 1.3205667282817466
- link link3: mass 1.2285446023550037 -> 1.0432921141432132
Joints:
- joint joint3: origin xyz=0.18711102593640605 0 -0.039 rpy=0 0 0 -> xyz=0.19979758594052155 0 -0.039 rpy=0 0 0
- joint joint4: origin xyz=0.30938949326204396 0 0.039 rpy=0 0 -3.14159265358979 -> xyz=0.16379979779976328 0 0.039 rpy=0 0 -3.14159265358979

Commit message: 20240415_60000dqn_ver3

File: dynamics/src/dynamics/urdf/single_arm_v22_19cm.urdf (robot description, URDF)
Before this commit: robot single_arm_v22_19cm, 8 links, 7 joints
Links:
- link link2: mass 1.3205667282817466 -> 1.544052439589766
- link link3: mass 1.0432921141432132 -> 1.1802522000406588
Joints:
- joint joint3: origin xyz=0.19979758594052155 0 -0.039 rpy=0 0 0 -> xyz=0.37543472292897284 0 -0.039 rpy=0 0 0
- joint joint4: origin xyz=0.16379979779976328 0 0.039 rpy=0 0 -3.14159265358979 -> xyz=0.2714365555500854 0 0.039 rpy=0 0 -3.14159265358979

File: dynamics/src/dynamics/urdf/single_arm_v22_19cm_motion.urdf (robot description, URDF)
Before this commit: robot single_arm_v22_19cm, 8 links, 7 joints
Links:
- link link2: mass 1.3205667282817466 -> 1.544052439589766
- link link3: mass 1.0432921141432132 -> 1.1802522000406588
Joints:
- joint joint3: origin xyz=0.19979758594052155 0 -0.039 rpy=0 0 0 -> xyz=0.37543472292897284 0 -0.039 rpy=0 0 0
- joint joint4: origin xyz=0.16379979779976328 0 0.039 rpy=0 0 -3.14159265358979 -> xyz=0.2714365555500854 0 0.039 rpy=0 0 -3.14159265358979

Commit message: 20240415cmd2_20240410-081152

File: dynamics/src/dynamics/urdf/single_arm_v22_19cm.urdf (robot description, URDF)
Before this commit: robot single_arm_v22_19cm, 8 links, 7 joints
Links:
- link link2: mass 1.544052439589766 -> 1.43173470539440
- link link3: mass 1.1802522000406588 -> 1.34744815174846
Joints:
- joint joint3: origin xyz=0.37543472292897284 0 -0.039 rpy=0 0 0 -> xyz=0.287164358118425 0 -0.039 rpy=0 0 0
- joint joint4: origin xyz=0.2714365555500854 0 0.039 rpy=0 0 -3.14159265358979 -> xyz=0.402835641881575 0 0.039 rpy=0 0 -3.14159265358979

File: dynamics/src/dynamics/urdf/single_arm_v22_19cm_motion.urdf (robot description, URDF)
Before this commit: robot single_arm_v22_19cm, 8 links, 7 joints
Links:
- link link2: mass 1.544052439589766 -> 1.43173470539440
- link link3: mass 1.1802522000406588 -> 1.34744815174846
Joints:
- joint joint3: origin xyz=0.37543472292897284 0 -0.039 rpy=0 0 0 -> xyz=0.287164358118425 0 -0.039 rpy=0 0 0
- joint joint4: origin xyz=0.2714365555500854 0 0.039 rpy=0 0 -3.14159265358979 -> xyz=0.402835641881575 0 0.039 rpy=0 0 -3.14159265358979
